Commit message: add config in myrobot_description

File: robot_description/myrobot_description/6dof/urdf/GEN3-6DOF_VISION_URDF_ARM_V01.urdf (robot description, URDF)
Before this commit: robot GEN3-6DOF_VISION_URDF_ARM_V01, 9 links, 8 joints
Links:
- link Base_Link: geometry collision mesh filename=package://myrobot_description/6dof/meshes/base_link.STL; visual mesh filename=package://myrobot_description/6dof/meshes/base_link.STL
- link Bicep_Link: geometry collision mesh filename=package://myrobot_description/6dof/meshes/bicep_link.STL; visual mesh filename=package://myrobot_description/6dof/meshes/bicep_link.STL
- link Bracelet_Link: geometry collision mesh filename=package://myrobot_description/6dof/meshes/bracelet_with_vis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; visual mesh filename=package://myrobot_description/6dof/meshes/bracelet_with_vis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
- link ForeArm_Link: geometry collision mesh filename=package://myrobot_description/6dof/meshes/forearm_link.STL; visual mesh filename=package://myrobot_description/6dof/meshes/forearm_link.STL
- link Shoulder_Link: geometry collision mesh filename=package://myrobot_description/6dof/meshes/shoulder_link.STL; visual mesh filename=package://myrobot_description/6dof/meshes/shoulder_link.STL
- link SphericalWrist1_Link: geometry collision mesh filename=package://myrobot_description/6dof/meshes/spherical_wrist_1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; visual mesh filename=package://myrobot_description/6dof/meshes/spherical_wrist_1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
- link SphericalWrist2_Link: geometry collision mesh filename=package://myrobot_description/6dof/meshes/spherical_wrist_2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; visual mesh filename=package://myrobot_description/6dof/meshes/spherical_wrist_2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
